File: board/easun-smp-telemetry.kicad_pcb (KiCad board)
At the start: 2 copper layers, 55 x 20 mm, 13 parts, among them J1 INVERTER, J2 PROG, U1 LM1117-3.3, U2 ESP32-C3-WROOM-02, U3 MAX3232 (SP3232E)

Commit message: WIP
Parts:
- added D1: LED, Connector_PinHeader_2.54mm:PinHeader_1x02_P2.54mm_Vertical, F.Cu at (136.0, 87.8)
- added R1: 270R, Resistor_SMD:R_0805_2012Metric_Pad1.20x1.40mm_HandSolder, F.Cu at (142.5, 88.0)
- moved C1 1.12 mm to (130.5, 94.0)
- moved J1 1.02 mm to (133.5, 91.0)
Connections:
- U2 pad 3: unconnected-(U2-GPIO4/ADC1_CH4) -> /LED
Routing:
- net /LED: track 0.00 -> 14.4 mm
- net Net-(R1-Pad2): track 0.00 -> 3.09 mm
- net /RX_INV: track 12.2 -> 10.9 mm
- net /TX_INV: track 14.6 -> 13.6 mm
