File: board/easun-smp-telemetry.kicad_pcb (KiCad board)
At the start: 2 copper layers, 55 x 20 mm, 15 parts, among them J1 INVERTER, J2 PROG, U1 LM1117-3.3, U2 ESP32-C3-WROOM-02, U3 MAX3232 (SP3232E)

Commit message: WIP
Parts:
- added C9: 1u, Capacitor_SMD:C_0805_2012Metric_Pad1.18x1.45mm_HandSolder, F.Cu at (154.5, 102.5)
- added R2: 10k, Resistor_SMD:R_0805_2012Metric_Pad1.20x1.40mm_HandSolder, F.Cu at (159.0, 102.5)
- U3: footprint Package_SO:SO-16_3.9x9.9mm_P1.27mm -> Package_SO:SOIC-16_3.9x9.9mm_P1.27mm
- moved C1 6.18 mm to (132.0, 88.0)
Connections:
- U2 pad 2: +3V3 -> Net-(U2-EN/CHIP_PU)
Routing:
- net +3V3: track 32.9 -> 72.5 mm, vias 15 -> 0
- net Net-(U2-EN/CHIP_PU): track 0.00 -> 17.6 mm
- net /VIN: track 12.7 -> 14.9 mm
- net /RX_ESP: track 28.5 -> 29.9 mm
- net /TX_ESP: track 30.6 -> 31.8 mm
- net /LED: track 14.4 -> 14.9 mm, vias 0 -> 2
- net GND: vias 0 -> 39
- added copper zone on B.Cu, net GND
- removed copper zone on B.Cu, net +3V3
Other:
- board text added: "easun-smp-telemetry v1.1"
- board text removed: "easun-smp-telemetry v1.0"
