File: board/easun-smp-telemetry.kicad_pcb (KiCad board)
At the start: 2 copper layers, 55 x 20 mm, 17 parts, among them J1 INVERTER, J2 PROG, U1 LM1117-3.3, U2 ESP32-C3-WROOM-02, U3 MAX3232 (SP3232E)

Commit message: WIP
Parts:
- moved U2 0.81 mm to (164.2, 91.3)
Routing:
- net +3V3: track 72.5 -> 77.3 mm
- net /LED: track 14.9 -> 18.6 mm
- net Net-(U2-EN/CHIP_PU): track 17.6 -> 20.0 mm
- net GND: vias 39 -> 40

Commit message: WIP
Parts:
- U2: footprint Espressif:ESP32-C3-WROOM-02 -> Drake:ESP32-C3-WROOM-02 Handsolder

Commit message: library update
Connections:
- U2 pad 3: /LED -> unconnected-(U2-GPIO4/ADC1_CH4-Pad3)
