File: board/easun-smp-telemetry.kicad_sch (KiCad schematic)
At the start: 13 parts, among them J1 INVERTER, J2 PROG, U1 LM1117-3.3, U2 ESP32-C3-WROOM-02, U3 MAX3232 (SP3232E)

Commit message: WIP
Parts:
- added D1: LED, Connector_PinHeader_2.54mm:PinHeader_1x02_P2.54mm_Vertical, symbol Device:LED
- added R1: 270R, Resistor_SMD:R_0805_2012Metric_Pad1.20x1.40mm_HandSolder, symbol Device:R
Connections:
- net GND: now also D1.1 (K)
- net LED: now reaches U2.3 (GPIO4/ADC1_CH4)
- net LED: now also R1.1
- new net: D1.2 (A), R1.2
- no-connect marks 15 -> 14
Changed lines of the file:
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@@
   (no_connect (at 74.93 146.05))
   (no_connect (at 125.73 50.8))
-  (no_connect (at 125.73 53.34))
   (no_connect (at 125.73 45.72))
   (no_connect (at 125.73 68.58))
@@
     (effects (font (size 1.27 1.27)) (justify right bottom))
   )
+  (label "LED" (at 213.36 93.98 180) (fields_autoplaced)
+    (effects (font (size 1.27 1.27)) (justify right bottom))
+  )
   (label "TX_INV" (at 227.33 60.96 180) (fields_autoplaced)
     (effects (font (size 1.27 1.27)) (justify right bottom))
@@
   (label "TX_INV" (at 115.57 151.13 0) (fields_autoplaced)
     (effects (font (size 1.27 1.27)) (justify left bottom))
+  )
+  (label "LED" (at 125.73 53.34 180) (fields_autoplaced)
+    (effects (font (size 1.27 1.27)) (justify right bottom))
   )
   (label "RX_INV" (at 115.57 140.97 0) (fields_autoplaced)
@@
   (symbol (lib_id "power:GND") (at 123.19 135.89 90) (unit 1)
     (in_bom yes) (on_board yes) (dnp no) (fields_autoplaced)
-    (property "Reference" "#PWR0103" (at 129.54 135.89 0)
+    (property "Reference" "#PWR0106" (at 129.54 135.89 0)
       (effects (font (size 1.27 1.27)) hide)
     )
@@
       (project "easun-smp-telemetry"
         (path "/32f9e9f8-9d15-4d51-acc1-705de5fd2b71"
-          (reference "#PWR0103") (unit 1) (value "GND") (footprint "")
+          (reference "#PWR0106") (unit 1) (value "GND") (footprint "")
         )
       )
@@
         (path "/32f9e9f8-9d15-4d51-acc1-705de5fd2b71"
           (reference "#PWR01") (unit 1) (value "+3V3") (footprint "")
+        )
+      )
+    )
+  )
+  (symbol (lib_id "Device:LED") (at 224.79 93.98 180) (unit 1)
+    (in_bom yes) (on_board yes) (dnp no) (fields_autoplaced)
+    (property "Reference" "D1" (at 226.3775 88.9889 0)
+      (effects (font (size 1.27 1.27)))
+    )
+    (property "Value" "LED" (at 226.3775 90.7511 0)
+      (effects (font (size 1.27 1.27)))
+    )
+    (property "Footprint" "Connector_PinHeader_2.54mm:PinHeader_1x02_P2.54mm_Vertical" (at 224.79 93.98 0)
+      (effects (font (size 1.27 1.27)) hide)
+    )
+    (property "Datasheet" "~" (at 224.79 93.98 0)
+      (effects (font (size 1.27 1.27)) hide)
+    )
+    (pin "1")
+    (pin "2")
+    (instances
+      (project "easun-smp-telemetry"
+        (path "/32f9e9f8-9d15-4d51-acc1-705de5fd2b71"
+          (reference "D1") (unit 1) (value "LED") (footprint "Connector_PinHeader_2.54mm:PinHeader_1x02_P2.54mm_Vertical")
         )
       )
@@
         (path "/32f9e9f8-9d15-4d51-acc1-705de5fd2b71"
           (reference "U1") (unit 1) (value "LM1117-3.3") (footprint "Package_TO_SOT_SMD:SOT-223-3_TabPin2")
+        )
+      )
+    )
+  )
+  (symbol (lib_id "Device:R") (at 217.17 93.98 90) (unit 1)
+    (in_bom yes) (on_board yes) (dnp no) (fields_autoplaced)
+    (property "Reference" "R1" (at 217.17 90.1319 90)
+      (effects (font (size 1.27 1.27)))
+    )
+    (property "Value" "270R" (at 217.17 91.8941 90)
+      (effects (font (size 1.27 1.27)))
+    )
+    (property "Footprint" "Resistor_SMD:R_0805_2012Metric_Pad1.20x1.40mm_HandSolder" (at 217.17 95.758 90)
+      (effects (font (size 1.27 1.27)) hide)
+    )
+    (property "Datasheet" "~" (at 217.17 93.98 0)
+      (effects (font (size 1.27 1.27)) hide)
+    )
+    (pin "1")
+    (pin "2")
+    (instances
+      (project "easun-smp-telemetry"
+        (path "/32f9e9f8-9d15-4d51-acc1-705de5fd2b71"
+          (reference "R1") (unit 1) (value "270R") (footprint "Resistor_SMD:R_0805_2012Metric_Pad1.20x1.40mm_HandSolder")
         )
       )
@@
         )
       )
+    )
+  )
+  (symbol (lib_id "power:GND") (at 228.6 93.98 90) (unit 1)
+    (in_bom yes) (on_board yes) (dnp no) (fields_autoplaced)
+    (property "Reference" "#PWR0105" (at 234.95 93.98 0)
+      (effects (font (size 1.27 1.27)) hide)
+    )
+    (property "Value" "GND" (at 231.775 94.2666 90)
+      (effects (font (size 1.27 1.27)) (justify right))
+    )
+    (property "Footprint" "" (at 228.6 93.98 0)
+      (effects (font (size 1.27 1.27)) hide)
+    )
+    (property "Datasheet" "" (at 228.6 93.98 0)
+      (effects (font (size 1.27 1.27)) hide)
+    )
+    (pin "1")
+    (instances
+      (project "easun-smp-telemetry"
+        (path "/32f9e9f8-9d15-4d51-acc1-705de5fd2b71"
+          (reference "#PWR0105") (unit 1) (value "GND") (footprint "")
+        )
+      )

Commit message: WIP
Parts:
- added C14: 1u, Capacitor_SMD:C_0805_2012Metric_Pad1.18x1.45mm_HandSolder, symbol Device:C
- added R18: 10k, Resistor_SMD:R_0805_2012Metric_Pad1.20x1.40mm_HandSolder, symbol Device:R
- J1: symbol Connector:Conn_01x04_Male -> Connector:Conn_01x04_Pin
- J2: symbol Connector:Conn_01x03_Female -> Connector:Conn_01x03_Socket
- U1: symbol Regulator_Linear:LM1117-3.3 -> Regulator_Linear:LM1117MP-3.3
- U3: footprint Package_SO:SO-16_3.9x9.9mm_P1.27mm -> Package_SO:SOIC-16_3.9x9.9mm_P1.27mm
Connections:
- net +3V3: now also R18.1; no longer U2.2 (EN/CHIP_PU)
- net GND: now also C14.2
- new net: C14.1, R18.2, U2.2 (EN/CHIP_PU)

Commit message: WIP
Parts:
- U2: footprint Espressif:ESP32-C3-WROOM-02 -> Drake:ESP32-C3-WROOM-02 Handsolder
Changed lines of the file:
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@@
       (effects (font (size 1.27 1.27)))
     )
-    (property "Footprint" "Espressif:ESP32-C3-WROOM-02" (at 152.4 92.71 0)
+    (property "Footprint" "Drake:ESP32-C3-WROOM-02 Handsolder" (at 152.4 92.71 0)
       (effects (font (size 1.27 1.27)) hide)
     )

Commit message: library update
Parts:
- U2: footprint Drake:ESP32-C3-WROOM-02 Handsolder -> PCM_Espressif:ESP32-C3-WROOM-02
Other:
- moved on the sheet: C14, R18
